File: Hardware/PCB/PicoWeatherStation/PicoWeatherStation.kicad_pcb (KiCad board)
At the start: 2 copper layers, 99.2 x 73 mm, 78 parts, among them J1 TOUCH_PANEL, J2 LCD_BL, Q1 AO3400A, SW1 SW_PICO_RST, SW2 SW_PICO_RST, SW3 SW_PICO_RST, SW4 SW_PICO_RST, SW5 SW_PICO_RST, SW6 SW_PICO_RST, SW7 SW_PICO_RST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

Commit message: PCB: prepare for manufacturing
Parts:
- added R208: 100k, Resistor_SMD:R_0805_2012Metric_Pad1.20x1.40mm_HandSolder, B.Cu at (147.8, 65.2)
- moved R202 0.56 mm to (147.8, 67.1)
- moved R201 0.42 mm to (147.8, 69.0)
Connections:
- U1 pad 33: unconnected-(U1-Pad33) -> GND
Routing:
- net VDD: track 517.5 -> 519.4 mm
- net TOUCH_~{CS}: track 26.2 -> 27.9 mm
- net GND: vias 79 -> 84
Other:
- board text added: "Pico Weather Station Version: 1.0 Designed by Tamas Karpati in 2022 https://github.com/tomikaa87/pico-weather-station/"
